File: EXPERIMENTOS_ELN3/EXPERIMENTOS_ELN3.kicad_sch (KiCad schematic)
At the start: 51 parts, among them J1 Screw_Terminal_01x03, J12 MC Out1, J13 MC Out2, J14 Conn_01x07_Socket, J6 MC out, U1 TL084, U2 MC1496

Commit message: pcb finished
Parts:
- U2: footprint MC1496BPG:MC1496BPG -> Package_DIP:CERDIP-14_W7.62mm_SideBrazed_LongPads
- renumbered J1 to P1
Changed lines of the file:
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@@
 			)
 		)
-		(property "Footprint" "MC1496BPG:MC1496BPG"
+		(property "Footprint" "Package_DIP:CERDIP-14_W7.62mm_SideBrazed_LongPads"
 			(at 125.73 130.81 0)
 			(effects
@@
 		(dnp no)
 		(fields_autoplaced yes)
-		(property "Reference" "J1"
+		(property "Reference" "P1"
 			(at 267.97 134.6199 90)
 			(effects
@@
 			(project "EXPERIMENTOS_ELN3"
 				(path "/233e5c0c-a235-4d8c-b5ea-273737d0ab22"
-					(reference "J1")
-					(unit 1)
-				)
+					(reference "P1")
+					(unit 1)
+				)
