File: EXPERIMENTOS_ELN3/ExperimentoPLL.kicad_sch (KiCad schematic)
At the start: 12 parts, among them J2 Conn_01x04_Socket, J3 Conn_01x01_Pin, J4 Conn_01x01_Socket, J5 Conn_01x01_Socket, U3 4046, U4 4029

Commit message: pcb finished
Parts:
- removed D3: LED, symbol Device:LED
- removed J4, J5: Conn_01x01_Socket, Connector_PinSocket_2.54mm:PinSocket_1x01_P2.54mm_Vertical, symbol Connector:Conn_01x01_Socket
- removed R24: R_Small_US, symbol Device:R_Small_US
- added C16: 100n, Capacitor_THT:C_Rect_L9.0mm_W2.5mm_P7.50mm_MKT, symbol Device:C
- added C17: 68n, Capacitor_THT:C_Disc_D3.4mm_W2.1mm_P2.50mm, symbol Device:C
- added D4: LED, LED_THT:LED_D3.0mm, symbol Device:LED
- added J1: Output, Connector_PinHeader_2.54mm:PinHeader_1x01_P2.54mm_Vertical, symbol Connector:Conn_01x01_Pin
- added J4: F_select_out, Connector_PinHeader_2.54mm:PinHeader_1x01_P2.54mm_Vertical, symbol Connector:Conn_01x01_Pin
- added J7: Seletor, Connector_PinHeader_2.54mm:PinHeader_1x03_P2.54mm_Vertical, symbol Connector:Conn_01x03_Pin
- added R24, R27: 10k, Resistor_THT:R_Axial_DIN0207_L6.3mm_D2.5mm_P10.16mm_Horizontal, symbol Device:R_US
- added R25: 100k, Resistor_THT:R_Axial_DIN0207_L6.3mm_D2.5mm_P10.16mm_Horizontal, symbol Device:R_US
- added R26: 4k7, Resistor_THT:R_Axial_DIN0207_L6.3mm_D2.5mm_P10.16mm_Horizontal, symbol Device:R_US
- C15: value C -> 68n; footprint TestPoint:TestPoint_2Pads_Pitch5.08mm_Drill1.3mm -> Capacitor_THT:C_Disc_D3.8mm_W2.6mm_P2.50mm
- J2: value Conn_01x04_Socket -> F Select
- J3: value Conn_01x01_Pin -> Ref In
- renumbered C16 to C19, PWR to P2
Connections:
- net GND: now also C15.2, U3.5 (Inh), U4.1 (PE), U4.5 (Cin), R24.1, R27.2
- net VDC: now also U4.10 (U/D), U4.9 (B/D)
- net at U3.1 (PCP): now also D4.2 (A)
- net at U3.11 (R1): now also R24.2
- net at U3.13 (PC2): now also R25.1
- net at U3.14 (SigIn): now also C16.2
- net PC2: now reaches U3.3 (RefIn)
- net PC2: now also J7.2 (Pin_2)
- net OUT: now reaches U3.4 (FOUT)
- net OUT: now also U4.15 (CK), J1.1 (Pin_1), J7.1 (Pin_1)
- net at U3.6 (C1): now also C17.2
- net at U3.7 (C2): now also C17.1
- net at U3.9 (VCOin): now also R25.2, R26.1
- net at J3.1 (Pin_1): now also C16.1
- net at J2.1 (Pin_1): now also U4.6 (Q1)
- net at J2.2 (Pin_2): now also U4.11 (Q2)
- net at J2.3 (Pin_3): now also U4.14 (Q3)
- net at J2.4 (Pin_4): now also U4.2 (Q4)
- net at C15.1: now also R26.2
- new net: D4.1 (K), R27.1
- new net: J4.1 (Pin_1), J7.3 (Pin_3)
- no-connect marks 0 -> 9
Other:
- moved on the sheet: C15, C18, J2, J3, P2, U4
