File: harpia2/harpia2.kicad_pcb (KiCad board)
At the start: 2 copper layers, 28 parts, among them Q1 BC547, Q2 BC547, Q3 TIP42C, Q4 TIP42C, U1 ESP32-DEVKIT-V1, U4 LM7805_TO220

Commit message: layout changes in harpia PCB
Parts:
- removed H1, H2, H3, H4: MountingHole_Pad, MountingHole:MountingHole_3.2mm_M3_ISO7380_Pad
- removed LED_SYS1: LED, LED_THT:LED_D3.0mm_Clear
- removed the Q1 at (80.8, 27.3)
- removed Q2: BC547, Package_TO_SOT_THT:TO-92_HandSolder
- removed Q3: TIP42C, Package_TO_SOT_THT:TO-220-3_Horizontal_TabDown
- removed the R1 at (57.5, 25.7)
- removed the R2 at (57.5, 29.8)
- removed R4: 330R, Resistor_THT:R_Axial_DIN0207_L6.3mm_D2.5mm_P15.24mm_Horizontal
- removed R_SHUNT1: 0R22, Resistor_THT:R_Axial_DIN0614_L14.3mm_D5.7mm_P20.32mm_Horizontal
- added U5: ~, BATTERY_HOLDER:18650_BATTERY_HOLDER, F.Cu at (110.6, 88.9)
- Q1: renamed from Q4; footprint Package_TO_SOT_THT:TO-220-3_Horizontal_TabDown -> Package_TO_SOT_THT:TO-220-3_Vertical
- R1: renamed from RB1; value 3R -> 2R2
- U4: footprint Package_TO_SOT_THT:TO-220-3_Horizontal_TabDown -> Package_TO_SOT_THT:TO-220-3_Vertical
- moved Q1 203.3 mm to (232.8, 95.1), turned to -90 degrees
- moved U4 196.5 mm to (232.7, 109.7), turned to -90 degrees
- moved SWITCH_TERMINAL1 180.5 mm to (228.2, 86.7)
- moved R1 175.2 mm to (227.2, 79.6)
- moved SWITCH_TERMINAL2 171.7 mm to (219.6, 86.7)
- moved C2 154.9 mm to (226.4, 108.8), turned to 180 degrees
- moved C1 154.5 mm to (226.4, 101.1), turned to 180 degrees
- moved R2 149.7 mm to (177.5, 123.2), turned to 90 degrees
- moved LED_PWR1 125.7 mm to (177.5, 126.4), turned to -90 degrees
- moved U2 116.6 mm to (125.8, 130.1), turned to 180 degrees
- moved SD_CARD_SOCKET1 116.6 mm to (175.9, 87.1)
- moved U1 112.7 mm to (201.0, 104.5)
- moved U3 98.0 mm to (143.7, 116.7), turned to 90 degrees
- moved CONN_SERVO1 86.3 mm to (124.1, 88.1), turned to -90 degrees
- moved CONN_SERVO2 83.5 mm to (124.1, 96.7), turned to -90 degrees
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- renumbered R3 to R2
Connections:
- Q1 pad 3: Net-(Q3-B) -> Net-(Q1-E)
- R1 pad 1: Net-(Q3-E) -> Net-(Q1-E)
- R2 pad 2: Net-(Q1-C) (its old number) -> GND
- U1 pad 25: LED_SYS_PIN -> unconnected-(U1-D27-Pad25)
- VBATT_IN1 pad 1: Net-(Q3-E) -> Net-(Q1-E)
Routing:
- net GND: track 0.00 -> 332.8 mm
- net +5V: track 0.00 -> 287.5 mm, vias 0 -> 2
- net Net-(Q1-E): track 0.00 -> 179.8 mm
- net OUT_SERVO1: track 0.00 -> 111.8 mm
- net OUT_SERVO2: track 0.00 -> 108.0 mm
- net Net-(Q1-C): track 0.00 -> 100.2 mm
- net MOSI: track 0.00 -> 68.0 mm
- net I2C_SCL: track 0.00 -> 65.4 mm
- net I2C_SDA: track 0.00 -> 63.3 mm
- net Net-(Q1-B): track 0.00 -> 45.8 mm
- net SCK: track 0.00 -> 27.3 mm
- net CS: track 0.00 -> 26.5 mm
- net MISO: track 0.00 -> 24.7 mm
- net Net-(LED_PWR1-K): track 0.00 -> 3.20 mm
- added copper zone on B.Cu, net GND
Other:
- board outline added: 150 x 59.5 mm
- board text added: "+"
- board text added: "+5V"
- board text added: "-"
- board text added: "A"
- board text added: "CS"
- board text added: "DISSIPADOR"
- board text added: "F"
- board text added: "GND"
- board text added: "JUMPER +5V"
- board text added: "MISO"
- board text added: "MOSI"
- board text added: "SCK"
- board text added: "SERVO1"
- board text added: "SERVO2"
- board text added: "VCC"
