File: harpia2/harpia2.kicad_sch (KiCad schematic)
At the start: 28 parts, among them Q1 BC547, Q2 BC547, Q3 TIP42C, Q4 TIP42C, U1 ESP32-DEVKIT-V1, U4 LM7805_TO220

Commit message: layout changes in harpia PCB
Parts:
- removed H1, H2, H3, H4: MountingHole_Pad, MountingHole:MountingHole_3.2mm_M3_ISO7380_Pad, symbol Mechanical:MountingHole_Pad
- removed LED_SYS1: LED, LED_THT:LED_D3.0mm_Clear, symbol Device:LED
- removed Q1, Q2: BC547, Package_TO_SOT_THT:TO-92_HandSolder, symbol Transistor_BJT:BC547
- removed Q3: TIP42C, Package_TO_SOT_THT:TO-220-3_Horizontal_TabDown, symbol Transistor_BJT:TIP42C
- removed R1, R2: 10k, Resistor_THT:R_Axial_DIN0207_L6.3mm_D2.5mm_P15.24mm_Horizontal, symbol Device:R
- removed R4: 330R, Resistor_THT:R_Axial_DIN0207_L6.3mm_D2.5mm_P15.24mm_Horizontal, symbol Device:R
- removed R_SHUNT1: 0R22, Resistor_THT:R_Axial_DIN0614_L14.3mm_D5.7mm_P20.32mm_Horizontal, symbol Device:R
- added U5: ~, BATTERY_HOLDER:18650_BATTERY_HOLDER, symbol battery_holder:battery_holder_2x
- Q1: renamed from Q4; footprint Package_TO_SOT_THT:TO-220-3_Horizontal_TabDown -> Package_TO_SOT_THT:TO-220-3_Vertical
- R1: renamed from RB1; value 3R -> 2R2
- U1: footprint MODULE_ESP32_DEVKIT_V1:MODULE_ESP32_DEVKIT_V1 -> ESP32-DEVKIT-V1:MODULE_ESP32_DEVKIT_V1
- U4: footprint Package_TO_SOT_THT:TO-220-3_Horizontal_TabDown -> Package_TO_SOT_THT:TO-220-3_Vertical
- renumbered R3 to R2
Connections:
- net GND: now also R2.2
- net at Q1.3 (E): now also R1.1, VBATT_IN1.1 (Pin_1)
- net LED_SYS_PIN: no longer names the net of U1.25 (D27)
- no-connect marks 27 -> 28
Other:
- moved on the sheet: LED_PWR1, R1, R2, U1, VBATT_IN1
